File: Kicad/mech_Keyboard.kicad_pcb (KiCad board)
At the start: 2 copper layers, 252.4 x 81 mm, 81 parts, among them SW1 SW_Push

Commit message: troubleshooting
Parts:
- moved REF** 19.2 mm to (175.8, 143.0)
- moved REF** 19.1 mm to (118.7, 143.0)
- moved REF** 1.11 mm to (194.1, 104.8)
- moved REF** 1.01 mm to (232.1, 123.9)
- moved REF** 0.93 mm to (213.1, 123.8)
- moved REF** 0.93 mm to (251.1, 104.8)
- moved REF** 0.79 mm to (251.3, 123.9)
- moved REF** 0.68 mm to (213.3, 104.8)
- moved REF** 0.67 mm to (232.4, 104.8)
- moved REF** 0.62 mm to (194.3, 123.7)
Routing:
- net COLUMN12: track 38.1 -> 163.7 mm, vias 0 -> 1
- net GND: track 43.9 -> 161.5 mm
- net COLUMN11: track 38.1 -> 138.7 mm
- net Net-(A1-3V3): track 29.5 -> 34.1 mm
- net COLUMN13: track 108.2 -> 107.3 mm
